Commit message: added aubo robots urdf.xacro

File: aubo_description/urdf/aubo.gazebo.xacro (robot description, xacro)
@@ -1,58 +1,64 @@
 <?xml version="1.0"?>
 <robot xmlns:xacro="http://www.ros.org/wiki/xacro">
-  <xacro:include filename="$(find aubo_description)/urdf/materials.xacro" />
   <xacro:macro name="aubo_arm_gazebo" params="prefix">
-     <!--base_Link-->
-     <gazebo reference = "${prefix}base_Link">
-	<material>Gazebo/Black</material>
-     </gazebo>
-     <!--shoulder_Link-->
-     <gazebo reference = "${prefix}shoulder_Link">
-	<material>Gazebo/Orange</material>
-     </gazebo>
-     <!--s_Link-->
-     <gazebo reference = "${prefix}s_Link">
-	<material>Gazebo/Black</material>
-     </gazebo>
-     <!--upperArm_Link-->
-     <gazebo reference = "${prefix}upperArm_Link">
-	<material>Gazebo/Orange</material>
-     </gazebo>
-     <!--f1_Link-->
-     <gazebo reference = "${prefix}f1_Link">
-	<material>Gazebo/Black</material>
-     </gazebo>
-     <!--foreArm_Link-->
-     <gazebo reference = "${prefix}foreArm_Link">
-	<material>Gazebo/Orange</material>
-     </gazebo>
-     <!--u_Link-->
-     <gazebo reference = "${prefix}u_Link">
-	<material>Gazebo/Black</material>
-     </gazebo>
-     <!--wrist1_Link-->
-     <gazebo reference = "${prefix}wrist1_Link">
-	<material>Gazebo/Orange</material>
-     </gazebo>
-     <!--w1_Link-->
-     <gazebo reference = "${prefix}w1_Link">
-	<material>Gazebo/Black</material>
-     </gazebo>
-     <!--wrist2_Link-->
-     <gazebo reference = "${prefix}wrist2_Link">
-	<material>Gazebo/Orange</material>
-     </gazebo>
-     <!--w2_Link-->
-     <gazebo reference = "${prefix}w2_Link">
-	<material>Gazebo/Black</material>
-     </gazebo>
-     <!--wrist3_Link-->
-     <gazebo reference = "${prefix}wrist3_Link">
-	<material>Gazebo/Black</material>
-     </gazebo>
-     <!--pedestal_Link-->
-     <gazebo reference = "${prefix}pedestal_Link">
-	<material>Gazebo/Green</material>
-     </gazebo>
+    <!--base_Link-->
+    <gazebo reference = "${prefix}base_Link">
+      <material>Gazebo/Black</material>
+    </gazebo>
+    <!--shoulder_Link-->
+    <gazebo reference = "${prefix}shoulder_Link">
+      <material>Gazebo/Orange</material>
+    </gazebo>
+    <!--s_Link-->
+    <gazebo reference = "${prefix}s_Link">
+      <material>Gazebo/Black</material>
+    </gazebo>
+    <!--upperArm_Link-->
+    <gazebo reference = "${prefix}upperArm_Link">
+      <material>Gazebo/Orange</material>
+    </gazebo>
+    <!--f1_Link-->
+    <gazebo reference = "${prefix}f1_Link">
+      <material>Gazebo/Black</material>
+    </gazebo>
+    <!--foreArm_Link-->
+    <gazebo reference = "${prefix}foreArm_Link">
+      <material>Gazebo/Orange</material>
+    </gazebo>
+    <!--u_Link-->
+    <gazebo reference = "${prefix}u_Link">
+      <material>Gazebo/Black</material>
+    </gazebo>
+    <!--wrist1_Link-->
+    <gazebo reference = "${prefix}wrist1_Link">
+      <material>Gazebo/Orange</material>
+    </gazebo>
+    <!--w1_Link-->
+    <gazebo reference = "${prefix}w1_Link">
+      <material>Gazebo/Black</material>
+    </gazebo>
+    <!--wrist2_Link-->
+    <gazebo reference = "${prefix}wrist2_Link">
+      <material>Gazebo/Orange</material>
+    </gazebo>
+    <!--w2_Link-->
+    <gazebo reference = "${prefix}w2_Link">
+      <material>Gazebo/Black</material>
+    </gazebo>
+    <!--wrist3_Link-->
+    <gazebo reference = "${prefix}wrist3_Link">
+      <material>Gazebo/Black</material>
+    </gazebo>
+    <!--pedestal_Link-->
+    <gazebo reference = "${prefix}pedestal_Link">
+      <material>Gazebo/Green</material>
+    </gazebo>
+    <gazebo>
+      <plugin name="ros_control" filename="libgazebo_ros_control.so">
+        <robotNamespace>/</robotNamespace>
+        <robotSimType>gazebo_ros_control/DefaultRobotHWSim</robotSimType>
+        <legacyModeNS>true</legacyModeNS>
+      </plugin>
+    </gazebo>
   </xacro:macro>
 </robot>

File: aubo_description/urdf/aubo.transmission.xacro (robot description, xacro)
@@ -1,9 +1,9 @@
 <?xml version="1.0"?>
 <robot xmlns:xacro="http://www.ros.org/wiki/xacro">
-  <xacro:macro name="aubo_arm_transmission" params="prefix">
+  <xacro:macro name="aubo_arm_transmission" params="prefix hardware_interface:=hardware_interface/EffortJointInterface">
     <transmission name="${prefix}shoulder_trans">
       <type>transmission_interface/SimpleTransmission</type>
       <joint name="${prefix}shoulder_joint">
-        <hardwareInterface>PositionJointInterface</hardwareInterface>
+        <hardwareInterface>${hardware_interface}</hardwareInterface>
       </joint>
       <actuator name="${prefix}shoulder_motor">
@@ -14,5 +14,5 @@
       <type>transmission_interface/SimpleTransmission</type>
       <joint name="${prefix}foreArm_joint">
-        <hardwareInterface>PositionJointInterface</hardwareInterface>
+        <hardwareInterface>${hardware_interface}</hardwareInterface>
       </joint>
       <actuator name="${prefix}foreArm_motor">
@@ -23,5 +23,5 @@
       <type>transmission_interface/SimpleTransmission</type>
       <joint name="${prefix}upperArm_joint">
-        <hardwareInterface>PositionJointInterface</hardwareInterface>
+        <hardwareInterface>${hardware_interface}</hardwareInterface>
       </joint>
       <actuator name="${prefix}upperArm_motor">
@@ -32,5 +32,5 @@
       <type>transmission_interface/SimpleTransmission</type>
       <joint name="${prefix}wrist1_joint">
-        <hardwareInterface>PositionJointInterface</hardwareInterface>
+        <hardwareInterface>${hardware_interface}</hardwareInterface>
       </joint>
       <actuator name="${prefix}wrist1_motor">
@@ -41,5 +41,5 @@
       <type>transmission_interface/SimpleTransmission</type>
       <joint name="${prefix}wrist2_joint">
-        <hardwareInterface>PositionJointInterface</hardwareInterface>
+        <hardwareInterface>${hardware_interface}</hardwareInterface>
       </joint>
       <actuator name="${prefix}wrist2_motor">
@@ -50,5 +50,5 @@
       <type>transmission_interface/SimpleTransmission</type>
       <joint name="${prefix}wrist3_joint">
-        <hardwareInterface>PositionJointInterface</hardwareInterface>
+        <hardwareInterface>${hardware_interface}</hardwareInterface>
       </joint>
       <actuator name="${prefix}wrist3_motor">

File: aubo_description/urdf/aubo_i10.urdf.xacro (robot description, xacro)
@@ -1,36 +1,36 @@
 <?xml version="1.0"?>
-<robot xmlns:xacro="http://www.ros.org/wiki/xacro" name="aubo_i5">
-  <xacro:macro name="aubo_i5" params="prefix">
+<robot xmlns:xacro="http://www.ros.org/wiki/xacro" name="aubo_i10">
+  <xacro:macro name="aubo_i10" params="prefix">
     <link name="${prefix}base_link">
       <visual>
         <origin xyz="0 0 0" rpy="0 0 0" />
         <geometry>
-          <mesh filename="package://aubo_description/meshes/aubo_i5/visual/base_link.DAE" />
-        </geometry>
-        <material name="">
-          <color rgba="1 1 1 1" />
-        </material>
-      </visual>
-      <collision>
-        <origin xyz="0 0 0" rpy="0 0 0" />
-        <geometry>
-          <mesh filename="package://aubo_description/meshes/aubo_i5/collision/base_link.STL" />
-        </geometry>
-      </collision>
-      <inertial>
-        <origin xyz="-1.4795E-13 0.0015384 0.020951" rpy="0 0 0" />
-        <mass value="0.83419" />
-        <inertia
-          ixx="0.0014414" ixy="7.8809E-15" ixz="8.5328E-16"
-          iyy="0.0013542" iyz="-1.4364E-05"
-          izz="0.0024659" />
+          <mesh filename="package://aubo_description/meshes/aubo_i10/base_link.DAE" />
+        </geometry>
+        <material name="">
+          <color rgba="1 1 1 1" />
+        </material>
+      </visual>
+      <collision>
+        <origin xyz="0 0 0" rpy="0 0 0" />
+        <geometry>
+          <mesh filename="package://aubo_description/meshes/aubo_i10/base_link.STL" />
+        </geometry>
+      </collision>
+      <inertial>
+        <origin xyz="-2.7535E-06 0.00054789 0.02299" rpy="0 0 0" />
+        <mass value="1.2345" />
+        <inertia
+          ixx="0.0029215" ixy="2.2046E-07" ixz="-3.4773E-08"
+          iyy="0.0028546" iyz="-7.6362E-06"
+          izz="0.0051176" />
       </inertial>
     </link>
     <joint name="${prefix}shoulder_joint" type="revolute">
-      <origin xyz="0 0 0.122" rpy="0 0 3.1416" />
+      <origin xyz="0 0 0.1632" rpy="-8.7138E-17 -4.3534E-32 3.1416" />
       <parent link="base_link" />
       <child link="shoulder_Link" />
       <axis xyz="0 0 1" />
-      <limit lower="-3.05" upper="3.05" velocity="2.62" effort="207.0"/>
+      <limit lower="-3.05" upper="3.05" effort="0" velocity="0" />
     </joint>
     <link name="${prefix}shoulder_Link">
@@ -38,31 +38,32 @@
         <origin xyz="0 0 0" rpy="0 0 0" />
         <geometry>
-          <mesh filename="package://aubo_description/meshes/aubo_i5/visual/shoulder_Link.DAE" />
-        </geometry>
-        <material name="">
-          <color rgba="1 1 1 1" />
-        </material>
-      </visual>
-      <collision>
-        <origin xyz="0 0 0" rpy="0 0 0" />
-        <geometry>
-          <mesh filename="package://aubo_description/meshes/aubo_i5/collision/shoulder_Link.STL" />
-        </geometry>
-      </collision>
-      <inertial>
-        <origin xyz="0.0 0.006 -0.002" rpy="0 0 0" />
-        <mass value="5.05" />
-        <inertia
-          ixx="0.0148" ixy="0" ixz="0"
-          iyy="0.0143" iyz="0"
-          izz="0.0095" />
+          <mesh
+            filename="package://aubo_description/meshes/aubo_i10/shoulder_Link.DAE" />
+        </geometry>
+        <material name="">
+          <color rgba="0.89804 0.91765 0.92941 1" />
+        </material>
+      </visual>
+      <collision>
+        <origin xyz="0 0 0" rpy="0 0 0" />
+        <geometry>
+          <mesh filename="package://aubo_description/meshes/aubo_i10/shoulder_Link.STL" />
+        </geometry>
+      </collision>
+      <inertial>
+        <origin xyz="0.00029287 0.14173 0.54281" rpy="0 0 0" />
+        <mass value="10.994" />
+        <inertia
+          ixx="2.2088" ixy="-0.00043922" ixz="-0.0025417"
+          iyy="2.1473" iyz="-0.049088"
+          izz="0.07998" />
       </inertial>
     </link>
     <joint name="${prefix}upperArm_joint" type="revolute">
-      <origin xyz="0 0.1215 0" rpy="-1.5708 -1.5708 0" />
+      <origin xyz="0 0.2013 0" rpy="-1.5708 -1.5708 0" />
       <parent link="shoulder_Link" />
       <child link="upperArm_Link" />
       <axis xyz="0 0 1" />
-      <limit lower="-3.05" upper="3.05" velocity="2.62" effort="207.0"/>
+      <limit lower="-3.05" upper="3.05" effort="0" velocity="0" />
     </joint>
     <link name="${prefix}upperArm_Link">
@@ -70,31 +71,31 @@
         <origin xyz="0 0 0" rpy="0 0 0" />
         <geometry>
-          <mesh filename="package://aubo_description/meshes/aubo_i5/visual/upperArm_Link.DAE" />
-        </geometry>
-        <material name="">
-          <color rgba="1 1 1 1" />
-        </material>
-      </visual>
-      <collision>
-        <origin xyz="0 0 0" rpy="0 0 0" />
-        <geometry>
-          <mesh filename="package://aubo_description/meshes/aubo_i5/collision/upperArm_Link.STL" />
-        </geometry>
-      </collision>
-      <inertial>
-        <origin xyz="0.304 0.0 -0.03" rpy="0 0 0" />
-        <mass value="11.90" />
-        <inertia
-          ixx="0.0305" ixy="0" ixz="0"
-          iyy="0.4505" iyz="0"
-          izz="0.0095" />
+          <mesh filename="package://aubo_description/meshes/aubo_i10/upperArm_Link.DAE" />
+        </geometry>
+        <material name="">
+          <color rgba="0.89804 0.91765 0.92941 1" />
+        </material>
+      </visual>
+      <collision>
+        <origin xyz="0 0 0" rpy="0 0 0" />
+        <geometry>
+          <mesh filename="package://aubo_description/meshes/aubo_i10/upperArm_Link.STL" />
+        </geometry>
+      </collision>
+      <inertial>
+        <origin xyz="0.31908 -3.7071E-06 -0.0042956" rpy="0 0 0" />
+        <mass value="5.3139" />
+        <inertia
+          ixx="0.0095171" ixy="7.2849E-06" ixz="-6.7014E-06"
+          iyy="0.11411" iyz="-1.1529E-06"
+          izz="0.11411" />
       </inertial>
     </link>
     <joint name="${prefix}foreArm_joint" type="revolute">
-      <origin xyz="0.408 0 0" rpy="-3.1416 -5.1632E-18 -5.459E-16" />
+      <origin xyz="0.647 0 0" rpy="3.1416 -4.5954E-17 -8.4328E-17" />
       <parent link="upperArm_Link" />
       <child link="foreArm_Link" />
       <axis xyz="0 0 1" />
-      <limit lower="-3.05" upper="3.05" velocity="2.62" effort="207.0"/>
+      <limit lower="-3.05" upper="3.05" effort="0" velocity="0" />
     </joint>
     <link name="${prefix}foreArm_Link">
@@ -102,31 +103,31 @@
         <origin xyz="0 0 0" rpy="0 0 0" />
         <geometry>
-          <mesh filename="package://aubo_description/meshes/aubo_i5/visual/foreArm_Link.DAE" />
-        </geometry>
-        <material name="">
-          <color rgba="1 1 1 1" />
-        </material>
-      </visual>
-      <collision>
-        <origin xyz="0 0 0" rpy="0 0 0" />
-        <geometry>
-          <mesh filename="package://aubo_description/meshes/aubo_i5/collision/foreArm_Link.STL" />
-        </geometry>
-      </collision>
-      <inertial>
-        <origin xyz="0.415 0.0 0.0992" rpy="0 0 0" />
-        <mass value="3.3" />
-        <inertia
-          ixx="0.0033" ixy="0" ixz="0.0009"
-          iyy="0.0575" iyz="0"
-          izz="0.0565" />
+          <mesh filename="package://aubo_description/meshes/aubo_i10/foreArm_Link.DAE" />
+        </geometry>
+        <material name="">
+          <color rgba="1 1 1 1" />
+        </material>
+      </visual>
+      <collision>
+        <origin xyz="0 0 0" rpy="0 0 0" />
+        <geometry>
+          <mesh filename="package://aubo_description/meshes/aubo_i10/foreArm_Link.STL" />
+        </geometry>
+      </collision>
+      <inertial>
+        <origin xyz="0.24431 6.6794E-06 0.12549" rpy="0 0 0" />
+        <mass value="3.1022" />
+        <inertia
+          ixx="0.0027288" ixy="-6.2713E-06" ixz="-0.0018082"
+          iyy="0.097825" iyz="3.5731E-07"
+          izz="0.097866" />
       </inertial>
     </link>
     <joint name="${prefix}wrist1_joint" type="revolute">
-      <origin xyz="0.376 0 0" rpy="3.1416 -1.8323E-15 1.5708" />
+      <origin xyz="0.6005 0 0" rpy="-3.1416 -1.4294E-15 1.5708" />
       <parent link="foreArm_Link" />
       <child link="wrist1_Link" />
       <axis xyz="0 0 1" />
-      <limit lower="-3.05" upper="3.05" velocity="3.14" effort="34.0"/>
+      <limit lower="-3.05" upper="3.05" effort="0" velocity="0" />
     </joint>
     <link name="${prefix}wrist1_Link">
@@ -134,31 +135,31 @@
         <origin xyz="0 0 0" rpy="0 0 0" />
         <geometry>
-          <mesh filename="package://aubo_description/meshes/aubo_i5/visual/wrist1_Link.DAE" />
-        </geometry>
-        <material name="">
-          <color rgba="1 1 1 1" />
-        </material>
-      </visual>
-      <collision>
-        <origin xyz="0 0 0" rpy="0 0 0" />
-        <geometry>
-          <mesh filename="package://aubo_description/meshes/aubo_i5/collision/wrist1_Link.STL" />
-        </geometry>
-      </collision>
-      <inertial>
-        <origin xyz="0. 0.028 -0.003" rpy="0 0 0" />
-        <mass value="1.62" />
-        <inertia
-          ixx="0.0023" ixy="0" ixz="0"
-          iyy="0.0013" iyz="0"
-          izz="0.0022" />
+          <mesh filename="package://aubo_description/meshes/aubo_i10/wrist1_Link.DAE" />
+        </geometry>
+        <material name="">
+          <color rgba="1 1 1 1" />
+        </material>
+      </visual>
+      <collision>
+        <origin xyz="0 0 0" rpy="0 0 0" />
+        <geometry>
+          <mesh filename="package://aubo_description/meshes/aubo_i10/wrist1_Link.STL" />
+        </geometry>
+      </collision>
+      <inertial>
+        <origin xyz="5.2305E-07 0.00026581 -0.0027894" rpy="0 0 0" />
+        <mass value="0.57981" />
+        <inertia
+          ixx="0.00088336" ixy="-6.425E-09" ixz="5.1594E-09"
+          iyy="0.00046118" iyz="-1.0734E-06"
+          izz="0.00085336" />
       </inertial>
     </link>
     <joint name="${prefix}wrist2_joint" type="revolute">
-      <origin xyz="0 0.1025 0" rpy="-1.5708 -1.8709E-15 -1.6653E-16" />
+      <origin xyz="0 0.1025 0" rpy="-1.5708 -7.0777E-16 -7.4101E-16" />
       <parent link="wrist1_Link" />
       <child link="wrist2_Link" />
       <axis xyz="0 0 1" />
-      <limit lower="-3.05" upper="3.05" velocity="3.14" effort="34.0"/>
+      <limit lower="-3.05" upper="3.05" effort="0" velocity="0" />
     </joint>
     <link name="${prefix}wrist2_Link">
@@ -166,31 +167,31 @@
         <origin xyz="0 0 0" rpy="0 0 0" />
         <geometry>
-          <mesh filename="package://aubo_description/meshes/aubo_i5/visual/wrist2_Link.DAE" />
-        </geometry>
-        <material name="">
-          <color rgba="1 1 1 1" />
-        </material>
-      </visual>
-      <collision>
-        <origin xyz="0 0 0" rpy="0 0 0" />
-        <geometry>
-          <mesh filename="package://aubo_description/meshes/aubo_i5/collision/wrist2_Link.STL" />
-        </geometry>
-      </collision>
-      <inertial>
-        <origin xyz="0. 0.0028 -0.003" rpy="0 0 0" />
-        <mass value="1.62" />
-        <inertia
-          ixx="0.0023" ixy="0" ixz="0"
-          iyy="0.0013" iyz="0"
-          izz="0.0022" />
+          <mesh filename="package://aubo_description/meshes/aubo_i10/wrist2_Link.DAE" />
+        </geometry>
+        <material name="">
+          <color rgba="1 1 1 1" />
+        </material>
+      </visual>
+      <collision>
+        <origin xyz="0 0 0" rpy="0 0 0" />
+        <geometry>
+          <mesh filename="package://aubo_description/meshes/aubo_i10/wrist2_Link.STL" />
+        </geometry>
+      </collision>
+      <inertial>
+        <origin xyz="-5.2305E-07 -0.00026581 -0.0027894" rpy="0 0 0" />
+        <mass value="0.57981" />
+        <inertia
+          ixx="0.00088336" ixy="-6.4251E-09" ixz="-5.1594E-09"
+          iyy="0.00046118" iyz="1.0734E-06"
+          izz="0.00085336" />
       </inertial>
     </link>
     <joint name="${prefix}wrist3_joint" type="revolute">
-      <origin xyz="0 -0.094 0" rpy="1.5708 0 1.7907E-15" />
+      <origin xyz="0 -0.094 0" rpy="1.5708 0 6.7283E-16" />
       <parent link="wrist2_Link" />
       <child link="wrist3_Link" />
       <axis xyz="0 0 1" />
-      <limit lower="-3.05" upper="3.05" velocity="3.14" effort="34.0"/>
+      <limit lower="-3.05" upper="3.05" effort="0" velocity="0" />
     </joint>
     <link name="${prefix}wrist3_Link">
@@ -198,23 +199,23 @@
         <origin xyz="0 0 0" rpy="0 0 0" />
         <geometry>
-          <mesh filename="package://aubo_description/meshes/aubo_i5/visual/wrist3_Link.DAE" />
-        </geometry>
-        <material name="">
-          <color rgba="1 1 1 1" />
-        </material>
-      </visual>
-      <collision>
-        <origin xyz="0 0 0" rpy="0 0 0" />
-        <geometry>
-          <mesh filename="package://aubo_description/meshes/aubo_i5/collision/wrist3_Link.STL" />
-        </geometry>
-      </collision>
-      <inertial>
-        <origin xyz="0.0 0.0 -0.0071" rpy="0 0 0" />
-        <mass value="0.15" />
-        <inertia
-          ixx="7.31376E-5" ixy="0" ixz="0"
-          iyy="7.19528E-5" iyz="0"
-          izz="0.00018" />
+          <mesh filename="package://aubo_description/meshes/aubo_i10/wrist3_Link.DAE" />
+        </geometry>
+        <material name="">
+          <color rgba="1 1 1 1" />
+        </material>
+      </visual>
+      <collision>
+        <origin xyz="0 0 0" rpy="0 0 0" />
+        <geometry>
+          <mesh filename="package://aubo_description/meshes/aubo_i10/wrist3_Link.STL" />
+        </geometry>
+      </collision>
+      <inertial>
+        <origin xyz="-2.2127E-09 0.00023722 -0.018629" rpy="0 0 0" />
+        <mass value="0.13669" />
+        <inertia
+          ixx="6.0946E-05" ixy="9.3663E-12" ixz="-1.3841E-12"
+          iyy="5.9501E-05" iyz="1.9944E-07"
+          izz="9.6981E-05" />
       </inertial>
     </link>

File: aubo_description/urdf/aubo_i3_robot.urdf.xacro (robot description, xacro)
@@ -1,5 +1,5 @@
 <?xml version="1.0"?>
-<robot xmlns:xacro="http://www.ros.org/wiki/xacro" name="aubo_i5">
-  <xacro:include filename="$(find aubo_description)/urdf/aubo_i5.urdf.xacro" />
+<robot xmlns:xacro="http://www.ros.org/wiki/xacro" name="aubo_i3">
+  <xacro:include filename="$(find aubo_description)/urdf/aubo_i3.urdf.xacro" />
   <xacro:include filename="$(find aubo_description)/urdf/common.gazebo.xacro" />
   <link name="world"/>
@@ -10,4 +10,6 @@
   </joint>
   <!-- Arm -->
-  <xacro:aubo_i5 prefix="" joint_limited="false"/>
+  <xacro:aubo_i3 prefix=""/>
+  <xacro:aubo_arm_transmission prefix=""/>
+  <xacro:aubo_arm_gazebo prefix=""/>
 </robot>

File: aubo_description/urdf/common.gazebo.xacro (robot description, xacro)
@@ -3,6 +3,7 @@
   <gazebo>
     <plugin name="ros_control" filename="libgazebo_ros_control.so">
-      <!--robotNamespace>/aubo_robot</robotNamespace-->
-      <!--robotSimType>gazebo_ros_control/DefaultRobotHWSim</robotSimType-->
+      <robotNamespace>/cubot</robotNamespace>
+      <robotSimType>gazebo_ros_control/DefaultRobotHWSim</robotSimType>
+      <legacyModeNS>true</legacyModeNS>
     </plugin>
   </gazebo>

File: aubo_description/urdf/materials.xacro (robot description, xacro)
@@ -2,20 +2,20 @@
 <robot xmlns:xacro="http://www.ros.org/wiki/xacro">
    <material name="black">
-	<color rgba="0.25098 0.25098 0.25098 1"/>
+	    <color rgba="0.25098 0.25098 0.25098 1"/>
    </material>
    <material name="orange">
-        <color rgba="${255/255} ${108/255} ${10/255} 1.0"/>
+      <color rgba="${255/255} ${108/255} ${10/255} 1.0"/>
    </material>
    <material name="white">
-        <color rgba="0.68627 0.69804 0.67451 1"/>
+      <color rgba="0.68627 0.69804 0.67451 1"/>
    </material>
    <material name="grey">
-        <color rgba="0.2 0.2 0.2 1.0"/>
+      <color rgba="0.2 0.2 0.2 1.0"/>
    </material>
    <material name="blue">
-        <color rgba="0.0 0.0 0.8 1.0"/>
+      <color rgba="0.0 0.0 0.8 1.0"/>
    </material>
    <material name="green">
-        <color rgba="0.0 0.8 0.0 1.0"/>
+      <color rgba="0.0 0.8 0.0 1.0"/>
    </material>
 </robot>
