Commit message: added aubo robots urdf.xacro

File: aubo_gazebo/urdf/aubo_i5.xacro (robot description, xacro)
@@ -1,4 +1,4 @@
 <?xml version="1.0"?>
-<robot name="aubo_i5" xmlns:xacro="http://ros.org/wiki/xacro">
+<robot xmlns:xacro="http://ros.org/wiki/xacro" name="aubo_i5">
  <!-- Defining the colors used in this robot -->
     <material name="Black">
@@ -21,112 +21,97 @@
     <!--/////////////////// DYNAMICS PARAM //////////////////////-->
     <xacro:macro name="I5_Shoulder_Inertia">
-        <origin xyz="0.0 0.006 -0.002"
-                rpy="0 0 0" />
+        <origin xyz="0.0 0.006 -0.002" rpy="0 0 0" />
         <mass value="5.05" />
-        <inertia ixx="0.0148"
-                 ixy="0"
-                 ixz="0"
-                 iyy="0.0143"
-                 iyz="-0.0"
-                 izz="0.0095" />
+        <inertia
+          ixx="0.0148" ixy="0" ixz="0"
+          iyy="0.0143" iyz="-0.0"
+          izz="0.0095" />
     </xacro:macro>
     <xacro:macro name="I5_UpperArm_Inertia">
-        <origin xyz="0.304 0.0 -0.03"
-                rpy="0 0 0" />
+        <origin xyz="0.304 0.0 -0.03" rpy="0 0 0" />
         <mass value="11.90" />
-        <inertia ixx="0.0305"
-                 ixy="0"
-                 ixz="0"
-                 iyy="0.4505"
-                 iyz="0"
-                 izz="0.0095" />
+        <inertia
+          ixx="0.0305" ixy="0" ixz="0"
+          iyy="0.4505" iyz="0"
+          izz="0.0095" />
     </xacro:macro>
     <xacro:macro name="I5_ForeArm_Inertia">
-        <origin xyz="0.415 0.0 0.0992"
-                rpy="0 0 0" />
-        <mass  value="3.3" />
-        <inertia ixx="0.0033"
-                 ixy="0"
-                 ixz="0.0009"
-                 iyy="0.0575"
-                 iyz="0"
-                 izz="0.0565" />
+        <origin xyz="0.415 0.0 0.0992" rpy="0 0 0" />
+        <mass value="3.3" />
+        <inertia
+          ixx="0.0033" ixy="0" ixz="0.0009"
+          iyy="0.0575" iyz="0"
+          izz="0.0565" />
     </xacro:macro>
     <xacro:macro name="I5_Wrist1_Inertia">
-        <origin xyz="0.0 0.0028 -0.003"
-                rpy="0 0 0" />
+        <origin xyz="0.0 0.0028 -0.003" rpy="0 0 0" />
         <mass value="1.62" />
-        <inertia ixx="0.0023"
-                 ixy="0"
-                 ixz="0"
-                 iyy="0.0013"
-                 iyz="0.0"
-                 izz="0.0022" />
+        <inertia
+          ixx="0.0023" ixy="0" ixz="0"
+          iyy="0.0013" iyz="0.0"
+          izz="0.0022" />
     </xacro:macro>
     <xacro:macro name="I5_Wrist2_Inertia">
-        <origin xyz="0.0 -0.0028 -0.003"
-                rpy="0 0 0" />
+        <origin xyz="0.0 -0.0028 -0.003" rpy="0 0 0" />
         <mass value="1.62" />
-        <inertia ixx="0.0023"
-                 ixy="0"
-                 ixz="0"
-                 iyy="0.0013"
-                 iyz="0.0"
-                 izz="0.0022" />
+        <inertia
+          ixx="0.0023" ixy="0" ixz="0"
+          iyy="0.0013" iyz="0.0"
+          izz="0.0022" />
     </xacro:macro>
     <xacro:macro name="I5_Wrist3_Inertia">
-        <origin xyz="0.0 0.0 -0.0071"
-                rpy="0 0 0" />
+        <origin xyz="0.0 0.0 -0.0071" rpy="0 0 0" />
         <mass value="0.40" />
-        <inertia ixx="0.013939"
-                 ixy="0"
-                 ixz="0"
-                 iyy="0.013988"
-                 iyz="0.0"
-                 izz="0.0224092" />
+        <inertia
+          ixx="0.013939" ixy="0" ixz="0"
+          iyy="0.013988" iyz="0.0"
+          izz="0.0224092" />
     </xacro:macro>
     <!--/////////////////////////////// BASE_LINK ////////////////////////////////////-->
    <link name="base_link">
+    <visual>
+      <origin xyz="0 0 0" rpy="0 0 0" />
+      <geometry>
+        <mesh filename="package://aubo_description/meshes/aubo_i5/visual/base_link.DAE" />
+      </geometry>
+      <material name="">
+        <color rgba="1 1 1 1" />
+      </material>
+    </visual>
+    <collision>
+      <origin xyz="0 0 0" rpy="0 0 0" />
+      <geometry>
+        <mesh filename="package://aubo_description/meshes/aubo_i5/collision/base_link.STL" />
+      </geometry>
+    </collision>
     <inertial>
       <origin xyz="-1.4795E-13 0.0015384 0.020951" rpy="0 0 0" />
       <mass value="0.83419" />
-      <inertia ixx="0.0014414" ixy="7.8809E-15" ixz="8.5328E-16" iyy="0.0013542" iyz="-1.4364E-05" izz="0.0024659" />
-    </inertial>
-    <visual>
-      <origin xyz="0 0 0" rpy="0 0 0" />
-      <geometry>
-        <mesh filename="package://aubo_description/meshes/aubo_i5/visual/base_link.DAE" />
-      </geometry>
-      <material name="">
-        <color rgba="1 1 1 1" />
-      </material>
-    </visual>
-    <collision>
-      <origin xyz="0 0 0" rpy="0 0 0" />
-      <geometry>
-        <mesh filename="package://aubo_description/meshes/aubo_i5/collision/base_link.STL" />
-      </geometry>
-    </collision>
+      <inertia
+        ixx="0.0014414" ixy="7.8809E-15" ixz="8.5328E-16"
+        iyy="0.0013542" iyz="-1.4364E-05"
+        izz="0.0024659" />
+    </inertial>
   </link>
   <!--/////////////////////////////// SHOULDER_LINK ////////////////////////////////////-->
   <link name="shoulder_Link">
+    <visual>
+      <origin xyz="0 0 0" rpy="0 0 0" />
+      <geometry>
+        <mesh filename="package://aubo_description/meshes/aubo_i5/visual/shoulder_Link.DAE" />
+      </geometry>
+      <material name="">
+        <color rgba="1 1 1 1" />
+      </material>
+    </visual>
+    <collision>
+      <origin xyz="0 0 0" rpy="0 0 0" />
+      <geometry>
+        <mesh filename="package://aubo_description/meshes/aubo_i5/collision/shoulder_Link.STL" />
+      </geometry>
+    </collision>
     <inertial>
       <xacro:I5_Shoulder_Inertia />
     </inertial>
-    <visual>
-      <origin xyz="0 0 0" rpy="0 0 0" />
-      <geometry>
-        <mesh filename="package://aubo_description/meshes/aubo_i5/visual/shoulder_Link.DAE" />
-      </geometry>
-      <material name="">
-        <color rgba="1 1 1 1" />
-      </material>
-    </visual>
-    <collision>
-      <origin xyz="0 0 0" rpy="0 0 0" />
-      <geometry>
-        <mesh filename="package://aubo_description/meshes/aubo_i5/collision/shoulder_Link.STL" />
-      </geometry>
-    </collision>
   </link>
   <!--/////////////////////////////// SHOULDER_JOINT ////////////////////////////////////-->
@@ -140,22 +125,22 @@
   <!--/////////////////////////////// UPPERARM_LINK ////////////////////////////////////-->
   <link name="upperArm_Link">
+    <visual>
+      <origin xyz="0 0 0" rpy="0 0 0" />
+      <geometry>
+        <mesh filename="package://aubo_description/meshes/aubo_i5/visual/upperArm_Link.DAE" />
+      </geometry>
+      <material name="">
+        <color rgba="1 1 1 1" />
+      </material>
+    </visual>
+    <collision>
+      <origin xyz="0 0 0" rpy="0 0 0" />
+      <geometry>
+        <mesh filename="package://aubo_description/meshes/aubo_i5/collision/upperArm_Link.STL" />
+      </geometry>
+    </collision>
     <inertial>
       <xacro:I5_UpperArm_Inertia />
     </inertial>
-    <visual>
-      <origin xyz="0 0 0" rpy="0 0 0" />
-      <geometry>
-        <mesh filename="package://aubo_description/meshes/aubo_i5/visual/upperArm_Link.DAE" />
-      </geometry>
-      <material name="">
-        <color rgba="1 1 1 1" />
-      </material>
-    </visual>
-    <collision>
-      <origin xyz="0 0 0" rpy="0 0 0" />
-      <geometry>
-        <mesh filename="package://aubo_description/meshes/aubo_i5/collision/upperArm_Link.STL" />
-      </geometry>
-    </collision>
   </link>
   <!--/////////////////////////////// UPPERARM_JOINT ////////////////////////////////////-->
@@ -169,22 +154,22 @@
   <!--/////////////////////////////// FOREARM_LINK ////////////////////////////////////-->
   <link name="foreArm_Link">
+    <visual>
+      <origin xyz="0 0 0" rpy="0 0 0" />
+      <geometry>
+        <mesh filename="package://aubo_description/meshes/aubo_i5/visual/foreArm_Link.DAE" />
+      </geometry>
+      <material name="">
+        <color rgba="1 1 1 1" />
+      </material>
+    </visual>
+    <collision>
+      <origin xyz="0 0 0" rpy="0 0 0" />
+      <geometry>
+        <mesh filename="package://aubo_description/meshes/aubo_i5/collision/foreArm_Link.STL" />
+      </geometry>
+    </collision>
     <inertial>
       <xacro:I5_ForeArm_Inertia />
     </inertial>
-    <visual>
-      <origin xyz="0 0 0" rpy="0 0 0" />
-      <geometry>
-        <mesh filename="package://aubo_description/meshes/aubo_i5/visual/foreArm_Link.DAE" />
-      </geometry>
-      <material name="">
-        <color rgba="1 1 1 1" />
-      </material>
-    </visual>
-    <collision>
-      <origin xyz="0 0 0" rpy="0 0 0" />
-      <geometry>
-        <mesh filename="package://aubo_description/meshes/aubo_i5/collision/foreArm_Link.STL" />
-      </geometry>
-    </collision>
   </link>
   <!--/////////////////////////////// FOREARM_JOINT ////////////////////////////////////-->
@@ -198,22 +183,22 @@
   <!--/////////////////////////////// WRIST1_LINK ////////////////////////////////////-->
   <link name="wrist1_Link">
+    <visual>
+      <origin xyz="0 0 0" rpy="0 0 0" />
+      <geometry>
+        <mesh filename="package://aubo_description/meshes/aubo_i5/visual/wrist1_Link.DAE" />
+      </geometry>
+      <material name="">
+        <color rgba="1 1 1 1" />
+      </material>
+    </visual>
+    <collision>
+      <origin xyz="0 0 0" rpy="0 0 0" />
+      <geometry>
+        <mesh filename="package://aubo_description/meshes/aubo_i5/collision/wrist1_Link.STL" />
+      </geometry>
+    </collision>
     <inertial>
       <xacro:I5_Wrist1_Inertia />
     </inertial>
-    <visual>
-      <origin xyz="0 0 0" rpy="0 0 0" />
-      <geometry>
-        <mesh filename="package://aubo_description/meshes/aubo_i5/visual/wrist1_Link.DAE" />
-      </geometry>
-      <material name="">
-        <color rgba="1 1 1 1" />
-      </material>
-    </visual>
-    <collision>
-      <origin xyz="0 0 0" rpy="0 0 0" />
-      <geometry>
-        <mesh filename="package://aubo_description/meshes/aubo_i5/collision/wrist1_Link.STL" />
-      </geometry>
-    </collision>
   </link>
   <!--/////////////////////////////// WRIST1_JOINT ////////////////////////////////////-->
@@ -227,22 +212,22 @@
   <!--/////////////////////////////// WRIST2_LINK ////////////////////////////////////-->
   <link name="wrist2_Link">
+    <visual>
+      <origin xyz="0 0 0" rpy="0 0 0" />
+      <geometry>
+        <mesh filename="package://aubo_description/meshes/aubo_i5/visual/wrist2_Link.DAE" />
+      </geometry>
+      <material name="">
+        <color rgba="1 1 1 1" />
+      </material>
+    </visual>
+    <collision>
+      <origin xyz="0 0 0" rpy="0 0 0" />
+      <geometry>
+        <mesh filename="package://aubo_description/meshes/aubo_i5/collision/wrist2_Link.STL" />
+      </geometry>
+    </collision>
     <inertial>
       <xacro:I5_Wrist2_Inertia />
     </inertial>
-    <visual>
-      <origin xyz="0 0 0" rpy="0 0 0" />
-      <geometry>
-        <mesh filename="package://aubo_description/meshes/aubo_i5/visual/wrist2_Link.DAE" />
-      </geometry>
-      <material name="">
-        <color rgba="1 1 1 1" />
-      </material>
-    </visual>
-    <collision>
-      <origin xyz="0 0 0" rpy="0 0 0" />
-      <geometry>
-        <mesh filename="package://aubo_description/meshes/aubo_i5/collision/wrist2_Link.STL" />
-      </geometry>
-    </collision>
   </link>
   <!--/////////////////////////////// WRIST2_JOINT ////////////////////////////////////-->
@@ -256,22 +241,22 @@
   <!--/////////////////////////////// WRIST3_LINK ////////////////////////////////////-->
   <link name="wrist3_Link">
+    <visual>
+      <origin xyz="0 0 0" rpy="0 0 0" />
+      <geometry>
+        <mesh filename="package://aubo_description/meshes/aubo_i5/visual/wrist3_Link.DAE" />
+      </geometry>
+      <material name="">
+        <color rgba="1 1 1 1" />
+      </material>
+    </visual>
+    <collision>
+      <origin xyz="0 0 0" rpy="0 0 0" />
+      <geometry>
+        <mesh filename="package://aubo_description/meshes/aubo_i5/collision/wrist3_Link.STL" />
+      </geometry>
+    </collision>
     <inertial>
       <xacro:I5_Wrist3_Inertia />
     </inertial>
-    <visual>
-      <origin xyz="0 0 0" rpy="0 0 0" />
-      <geometry>
-        <mesh filename="package://aubo_description/meshes/aubo_i5/visual/wrist3_Link.DAE" />
-      </geometry>
-      <material name="">
-        <color rgba="1 1 1 1" />
-      </material>
-    </visual>
-    <collision>
-      <origin xyz="0 0 0" rpy="0 0 0" />
-      <geometry>
-        <mesh filename="package://aubo_description/meshes/aubo_i5/collision/wrist3_Link.STL" />
-      </geometry>
-    </collision>
   </link>
   <!--/////////////////////////////// WRIST3_JOINT ////////////////////////////////////-->
@@ -312,6 +297,5 @@
        <type>transmission_interface/SimpleTransmission</type>
        <joint name="${joint_name}">
-         <!--<hardwareInterface>hardware_interface/PositionJointInterface</hardwareInterface>-->
-         <hardwareInterface>hardware_interface/PositionJointInterface</hardwareInterface>
+         <hardwareInterface>hardware_interface/EffortJointInterface</hardwareInterface>
        </joint>
        <actuator name="${joint_name}_motor">
@@ -328,7 +312,8 @@
   <!-- ros_control plugin -->
   <gazebo>
-      <plugin name="gazebo_ros_control" filename="libgazebo_ros_control.so">
-          <robotNamespace>/aubo_i5</robotNamespace>
-      </plugin>
+    <plugin name="gazebo_ros_control" filename="libgazebo_ros_control.so">
+      <robotNamespace>/aubo_i5</robotNamespace>
+      <legacyModeNS>True</legacyModeNS>
+    </plugin>
   </gazebo>
 </robot>
