Commit message: add private node capabilities

File: aubo_description/urdf/aubo.transmission.xacro (robot description, xacro)
@@ -1,5 +1,6 @@
 <?xml version="1.0"?>
 <robot xmlns:xacro="http://www.ros.org/wiki/xacro">
-  <xacro:macro name="aubo_arm_transmission" params="prefix hardware_interface:=hardware_interface/EffortJointInterface">
+  <xacro:macro name="aubo_arm_transmission"
+    params="prefix hardware_interface:=hardware_interface/EffortJointInterface">
     <transmission name="${prefix}shoulder_trans">
       <type>transmission_interface/SimpleTransmission</type>

File: aubo_description/urdf/aubo_i3_robot.urdf.xacro (robot description, xacro)
@@ -3,4 +3,5 @@
   <xacro:include filename="$(find aubo_description)/urdf/aubo_i3.urdf.xacro" />
   <xacro:include filename="$(find aubo_description)/urdf/common.gazebo.xacro" />
+  <!-- World -->
   <link name="world"/>
   <joint name="world_joint" type="fixed">

File: aubo_description/urdf/aubo_i5_robot.urdf.xacro (robot description, xacro)
@@ -3,4 +3,5 @@
   <xacro:include filename="$(find aubo_description)/urdf/aubo_i5.urdf.xacro" />
   <xacro:include filename="$(find aubo_description)/urdf/common.gazebo.xacro" />
+  <!-- World -->
   <link name="world"/>
   <joint name="world_joint" type="fixed">
@@ -10,4 +11,4 @@
   </joint>
   <!-- Arm -->
-  <xacro:aubo_i5 prefix="" joint_limited="false"/>
+  <xacro:aubo_i5 prefix=""/>
 </robot>
