Commit message: added install targets

File: aubo_description/urdf/aubo_i5_robot.urdf.xacro (robot description, xacro)
@@ -5,10 +5,10 @@
   <!-- World -->
   <link name="world"/>
-  <joint name="world_joint" type="fixed">
+  <!-- Arm -->
+  <joint name="base_joint" type="fixed">
+    <origin xyz="0 0 0" rpy="0 0 0"/>
     <parent link="world"/>
     <child link = "base_link"/>
-    <origin xyz="0 0 0" rpy="0 0 0"/>
   </joint>
-  <!-- Arm -->
   <xacro:aubo_i5 prefix=""/>
 </robot>
