Commit message: implemented aubo_i5 joint limits in urdf

File: aubo_description/urdf/aubo_i5.urdf.xacro (robot description, xacro)
@@ -1,5 +1,10 @@
-<?xml version="1.0"?>
 <robot xmlns:xacro="http://www.ros.org/wiki/xacro" name="aubo_i5">
-  <xacro:macro name="aubo_i5" params="prefix">
+  <xacro:macro name="aubo_i5" params="prefix
+    shoulder_joint_min:=-3.05 shoulder_joint_max:=3.05
+    upperArm_joint_min:=-3.05 upperArm_joint_max:=3.05
+    foreArm_joint_min:=-3.05  foreArm_joint_max:=3.05
+    wrist1_joint_min:=-3.05   wrist1_joint_max:=3.05
+    wrist2_joint_min:=-3.05   wrist2_joint_max:=3.05
+    wrist3_joint_min:=-3.05   wrist3_joint_max:=3.05">
     <link name="${prefix}base_link">
       <visual>
@@ -32,5 +37,5 @@
       <child link="shoulder_Link" />
       <axis xyz="0 0 1" />
-      <limit lower="-3.05" upper="3.05" velocity="2.62" effort="207.0"/>
+      <limit lower="${shoulder_joint_min}" upper="${shoulder_joint_max}" velocity="2.62" effort="207.0"/>
     </joint>
     <link name="${prefix}shoulder_Link">
@@ -64,5 +69,5 @@
       <child link="upperArm_Link" />
       <axis xyz="0 0 1" />
-      <limit lower="-3.05" upper="3.05" velocity="2.62" effort="207.0"/>
+      <limit lower="${upperArm_joint_min}" upper="${upperArm_joint_max}" velocity="2.62" effort="207.0"/>
     </joint>
     <link name="${prefix}upperArm_Link">
@@ -96,5 +101,5 @@
       <child link="foreArm_Link" />
       <axis xyz="0 0 1" />
-      <limit lower="-3.05" upper="3.05" velocity="2.62" effort="207.0"/>
+      <limit lower="${foreArm_joint_min}" upper="${foreArm_joint_max}" velocity="2.62" effort="207.0"/>
     </joint>
     <link name="${prefix}foreArm_Link">
@@ -128,5 +133,5 @@
       <child link="wrist1_Link" />
       <axis xyz="0 0 1" />
-      <limit lower="-3.05" upper="3.05" velocity="3.14" effort="34.0"/>
+      <limit lower="${wrist1_joint_min}" upper="${wrist1_joint_max}" velocity="3.14" effort="34.0"/>
     </joint>
     <link name="${prefix}wrist1_Link">
@@ -160,5 +165,5 @@
       <child link="wrist2_Link" />
       <axis xyz="0 0 1" />
-      <limit lower="-3.05" upper="3.05" velocity="3.14" effort="34.0"/>
+      <limit lower="${wrist2_joint_min}" upper="${wrist2_joint_max}" velocity="3.14" effort="34.0"/>
     </joint>
     <link name="${prefix}wrist2_Link">
@@ -192,5 +197,5 @@
       <child link="wrist3_Link" />
       <axis xyz="0 0 1" />
-      <limit lower="-3.05" upper="3.05" velocity="3.14" effort="34.0"/>
+      <limit lower="${wrist3_joint_min}" upper="${wrist3_joint_max}" velocity="3.14" effort="34.0"/>
     </joint>
     <link name="${prefix}wrist3_Link">

Commit message: code clean up

File: aubo_description/urdf/aubo_i5.urdf.xacro (robot description, xacro)
@@ -1,2 +1,3 @@
+<?xml version="1.0"?>
 <robot xmlns:xacro="http://www.ros.org/wiki/xacro" name="aubo_i5">
   <xacro:macro name="aubo_i5" params="prefix
@@ -33,5 +34,5 @@
     </link>
     <joint name="${prefix}shoulder_joint" type="revolute">
-      <origin xyz="0 0 0.122" rpy="0 0 3.1416" />
+      <origin xyz="0 0 0.122" rpy="0 0 ${pi}" />
       <parent link="base_link" />
       <child link="shoulder_Link" />
@@ -65,5 +66,5 @@
     </link>
     <joint name="${prefix}upperArm_joint" type="revolute">
-      <origin xyz="0 0.1215 0" rpy="-1.5708 -1.5708 0" />
+      <origin xyz="0 0.1215 0" rpy="${-pi/2} ${-pi/2} 0" />
       <parent link="shoulder_Link" />
       <child link="upperArm_Link" />
@@ -97,5 +98,5 @@
     </link>
     <joint name="${prefix}foreArm_joint" type="revolute">
-      <origin xyz="0.408 0 0" rpy="-3.1416 -5.1632E-18 -5.459E-16" />
+      <origin xyz="0.408 0 0" rpy="${-pi} 0 0" />
       <parent link="upperArm_Link" />
       <child link="foreArm_Link" />
@@ -129,5 +130,5 @@
     </link>
     <joint name="${prefix}wrist1_joint" type="revolute">
-      <origin xyz="0.376 0 0" rpy="3.1416 -1.8323E-15 1.5708" />
+      <origin xyz="0.376 0 0" rpy="${pi} 0 ${pi/2}" />
       <parent link="foreArm_Link" />
       <child link="wrist1_Link" />
@@ -161,5 +162,5 @@
     </link>
     <joint name="${prefix}wrist2_joint" type="revolute">
-      <origin xyz="0 0.1025 0" rpy="-1.5708 -1.8709E-15 -1.6653E-16" />
+      <origin xyz="0 0.1025 0" rpy="${-pi/2} 0 0" />
       <parent link="wrist1_Link" />
       <child link="wrist2_Link" />
@@ -193,5 +194,5 @@
     </link>
     <joint name="${prefix}wrist3_joint" type="revolute">
-      <origin xyz="0 -0.094 0" rpy="1.5708 0 1.7907E-15" />
+      <origin xyz="0 -0.094 0" rpy="${pi/2} 0 0" />
       <parent link="wrist2_Link" />
       <child link="wrist3_Link" />

Commit message: implemented aubo_i5 urdf calibration support

File: aubo_description/urdf/aubo_i5.urdf.xacro (robot description, xacro)
@@ -1,11 +1,12 @@
 <?xml version="1.0"?>
-<robot xmlns:xacro="http://www.ros.org/wiki/xacro" name="aubo_i5">
+<robot xmlns:xacro="http://www.ros.org/wiki/xacro">
   <xacro:macro name="aubo_i5" params="prefix
-    shoulder_joint_min:=-3.05 shoulder_joint_max:=3.05
-    upperArm_joint_min:=-3.05 upperArm_joint_max:=3.05
-    foreArm_joint_min:=-3.05  foreArm_joint_max:=3.05
-    wrist1_joint_min:=-3.05   wrist1_joint_max:=3.05
-    wrist2_joint_min:=-3.05   wrist2_joint_max:=3.05
-    wrist3_joint_min:=-3.05   wrist3_joint_max:=3.05">
+    *shoulder_calibration
+    *upperArm_calibration
+    *foreArm_calibration
+    *wrist1_calibration
+    *wrist2_calibration
+    *wrist3_calibration
+    *wrist3_limit">
     <link name="${prefix}base_link">
       <visual>
@@ -35,8 +36,9 @@
     <joint name="${prefix}shoulder_joint" type="revolute">
       <origin xyz="0 0 0.122" rpy="0 0 ${pi}" />
-      <parent link="base_link" />
-      <child link="shoulder_Link" />
-      <axis xyz="0 0 1" />
-      <limit lower="${shoulder_joint_min}" upper="${shoulder_joint_max}" velocity="2.62" effort="207.0"/>
+      <parent link="${prefix}base_link" />
+      <child link="${prefix}shoulder_Link" />
+      <axis xyz="0 0 1" />
+      <xacro:insert_block name="shoulder_calibration"/>
+      <limit lower="-3.05" upper="3.05" velocity="2.62" effort="207.0"/>
     </joint>
     <link name="${prefix}shoulder_Link">
@@ -67,8 +69,9 @@
     <joint name="${prefix}upperArm_joint" type="revolute">
       <origin xyz="0 0.1215 0" rpy="${-pi/2} ${-pi/2} 0" />
-      <parent link="shoulder_Link" />
-      <child link="upperArm_Link" />
-      <axis xyz="0 0 1" />
-      <limit lower="${upperArm_joint_min}" upper="${upperArm_joint_max}" velocity="2.62" effort="207.0"/>
+      <parent link="${prefix}shoulder_Link" />
+      <child link="${prefix}upperArm_Link" />
+      <axis xyz="0 0 1" />
+      <xacro:insert_block name="upperArm_calibration"/>
+      <limit lower="-3.05" upper="3.05" velocity="2.62" effort="207.0"/>
     </joint>
     <link name="${prefix}upperArm_Link">
@@ -99,8 +102,9 @@
     <joint name="${prefix}foreArm_joint" type="revolute">
       <origin xyz="0.408 0 0" rpy="${-pi} 0 0" />
-      <parent link="upperArm_Link" />
-      <child link="foreArm_Link" />
-      <axis xyz="0 0 1" />
-      <limit lower="${foreArm_joint_min}" upper="${foreArm_joint_max}" velocity="2.62" effort="207.0"/>
+      <parent link="${prefix}upperArm_Link" />
+      <child link="${prefix}foreArm_Link" />
+      <axis xyz="0 0 1" />
+      <xacro:insert_block name="foreArm_calibration"/>
+      <limit lower="-3.05" upper="3.05" velocity="2.62" effort="207.0"/>
     </joint>
     <link name="${prefix}foreArm_Link">
@@ -131,8 +135,9 @@
     <joint name="${prefix}wrist1_joint" type="revolute">
       <origin xyz="0.376 0 0" rpy="${pi} 0 ${pi/2}" />
-      <parent link="foreArm_Link" />
-      <child link="wrist1_Link" />
-      <axis xyz="0 0 1" />
-      <limit lower="${wrist1_joint_min}" upper="${wrist1_joint_max}" velocity="3.14" effort="34.0"/>
+      <parent link="${prefix}foreArm_Link" />
+      <child link="${prefix}wrist1_Link" />
+      <axis xyz="0 0 1" />
+      <xacro:insert_block name="wrist1_calibration"/>
+      <limit lower="-3.05" upper="3.05" velocity="3.14" effort="34.0"/>
     </joint>
     <link name="${prefix}wrist1_Link">
@@ -163,8 +168,9 @@
     <joint name="${prefix}wrist2_joint" type="revolute">
       <origin xyz="0 0.1025 0" rpy="${-pi/2} 0 0" />
-      <parent link="wrist1_Link" />
-      <child link="wrist2_Link" />
-      <axis xyz="0 0 1" />
-      <limit lower="${wrist2_joint_min}" upper="${wrist2_joint_max}" velocity="3.14" effort="34.0"/>
+      <parent link="${prefix}wrist1_Link" />
+      <child link="${prefix}wrist2_Link" />
+      <axis xyz="0 0 1" />
+      <xacro:insert_block name="wrist2_calibration"/>
+      <limit lower="-3.05" upper="3.05" velocity="3.14" effort="34.0"/>
     </joint>
     <link name="${prefix}wrist2_Link">
@@ -195,8 +201,9 @@
     <joint name="${prefix}wrist3_joint" type="revolute">
       <origin xyz="0 -0.094 0" rpy="${pi/2} 0 0" />
-      <parent link="wrist2_Link" />
-      <child link="wrist3_Link" />
-      <axis xyz="0 0 1" />
-      <limit lower="${wrist3_joint_min}" upper="${wrist3_joint_max}" velocity="3.14" effort="34.0"/>
+      <parent link="${prefix}wrist2_Link" />
+      <child link="${prefix}wrist3_Link" />
+      <axis xyz="0 0 1" />
+      <xacro:insert_block name="wrist3_calibration"/>
+      <xacro:insert_block name="wrist3_limit"/>
     </joint>
     <link name="${prefix}wrist3_Link">

File: aubo_description/urdf/aubo_i5_robot.urdf.xacro (robot description, xacro)
@@ -11,4 +11,12 @@
     <child link = "base_link"/>
   </joint>
-  <xacro:aubo_i5 prefix=""/>
+  <xacro:aubo_i5 prefix="">
+    <calibration rising="0.0"/>
+    <calibration rising="0.0"/>
+    <calibration rising="0.0"/>
+    <calibration rising="0.0"/>
+    <calibration rising="0.0"/>
+    <calibration rising="0.0"/>
+    <limit lower="-3.05" upper="3.05" velocity="3.14" effort="34.0"/>
+  </xacro:aubo_i5>
 </robot>

Commit message: implemented joints_offset parameter

File: aubo_description/urdf/aubo_i5.urdf.xacro (robot description, xacro)
@@ -1,5 +1,5 @@
 <?xml version="1.0"?>
 <robot xmlns:xacro="http://www.ros.org/wiki/xacro">
-  <xacro:macro name="aubo_i5" params="prefix
+  <xacro:macro name="aubo_i5" params="prefix:=''
     *shoulder_calibration
     *upperArm_calibration
