Commit message: general improvements

File: aubo_description/urdf/aubo_i10.urdf.xacro (robot description, xacro)
@@ -1,5 +1,6 @@
 <?xml version="1.0"?>
-<robot xmlns:xacro="http://www.ros.org/wiki/xacro" name="aubo_i10">
-  <xacro:macro name="aubo_i10" params="prefix">
+<robot xmlns:xacro="http://www.ros.org/wiki/xacro">
+  <xacro:macro name="aubo_i10" params="prefix:=''
+    *wrist3_limit">
     <link name="${prefix}base_link">
       <visual>
@@ -28,9 +29,9 @@
     </link>
     <joint name="${prefix}shoulder_joint" type="revolute">
-      <origin xyz="0 0 0.1632" rpy="-8.7138E-17 -4.3534E-32 3.1416" />
-      <parent link="base_link" />
-      <child link="shoulder_Link" />
-      <axis xyz="0 0 1" />
-      <limit lower="-3.05" upper="3.05" effort="0" velocity="0" />
+      <origin xyz="0. 0. 0.1632" rpy="0. 0. ${pi}"/>
+      <parent link="${prefix}base_link"/>
+      <child link="${prefix}shoulder_Link"/>
+      <axis xyz="0 0 1"/>
+      <limit lower="-3.05" upper="3.05" velocity="3.14" effort="207.0"/>
     </joint>
     <link name="${prefix}shoulder_Link">
@@ -61,9 +62,9 @@
     </link>
     <joint name="${prefix}upperArm_joint" type="revolute">
-      <origin xyz="0 0.2013 0" rpy="-1.5708 -1.5708 0" />
-      <parent link="shoulder_Link" />
-      <child link="upperArm_Link" />
-      <axis xyz="0 0 1" />
-      <limit lower="-3.05" upper="3.05" effort="0" velocity="0" />
+      <origin xyz="0. 0.2013 0." rpy="${-pi/2} ${-pi/2} 0"/>
+      <parent link="${prefix}shoulder_Link"/>
+      <child link="${prefix}upperArm_Link"/>
+      <axis xyz="0 0 1"/>
+      <limit lower="-3.05" upper="3.05" velocity="3.14" effort="207.0"/>
     </joint>
     <link name="${prefix}upperArm_Link">
@@ -93,9 +94,9 @@
     </link>
     <joint name="${prefix}foreArm_joint" type="revolute">
-      <origin xyz="0.647 0 0" rpy="3.1416 -4.5954E-17 -8.4328E-17" />
-      <parent link="upperArm_Link" />
-      <child link="foreArm_Link" />
-      <axis xyz="0 0 1" />
-      <limit lower="-3.05" upper="3.05" effort="0" velocity="0" />
+      <origin xyz="0.647 0. 0." rpy="${pi} 0. 0."/>
+      <parent link="${prefix}upperArm_Link"/>
+      <child link="${prefix}foreArm_Link"/>
+      <axis xyz="0 0 1"/>
+      <limit lower="-3.05" upper="3.05" velocity="2.62" effort="207.0"/>
     </joint>
     <link name="${prefix}foreArm_Link">
@@ -125,9 +126,9 @@
     </link>
     <joint name="${prefix}wrist1_joint" type="revolute">
-      <origin xyz="0.6005 0 0" rpy="-3.1416 -1.4294E-15 1.5708" />
-      <parent link="foreArm_Link" />
-      <child link="wrist1_Link" />
-      <axis xyz="0 0 1" />
-      <limit lower="-3.05" upper="3.05" effort="0" velocity="0" />
+      <origin xyz="0.6005 0. 0." rpy="${-pi} 0. ${pi/2}"/>
+      <parent link="${prefix}foreArm_Link"/>
+      <child link="${prefix}wrist1_Link"/>
+      <axis xyz="0 0 1"/>
+      <limit lower="-3.05" upper="3.05" velocity="3.14" effort="34.0"/>
     </joint>
     <link name="${prefix}wrist1_Link">
@@ -157,9 +158,9 @@
     </link>
     <joint name="${prefix}wrist2_joint" type="revolute">
-      <origin xyz="0 0.1025 0" rpy="-1.5708 -7.0777E-16 -7.4101E-16" />
-      <parent link="wrist1_Link" />
-      <child link="wrist2_Link" />
-      <axis xyz="0 0 1" />
-      <limit lower="-3.05" upper="3.05" effort="0" velocity="0" />
+      <origin xyz="0. 0.1025 0." rpy="${-pi/2} 0. 0."/>
+      <parent link="${prefix}wrist1_Link"/>
+      <child link="${prefix}wrist2_Link"/>
+      <axis xyz="0 0 1"/>
+      <limit lower="-3.05" upper="3.05" velocity="3.14" effort="34.0"/>
     </joint>
     <link name="${prefix}wrist2_Link">
@@ -189,9 +190,9 @@
     </link>
     <joint name="${prefix}wrist3_joint" type="revolute">
-      <origin xyz="0 -0.094 0" rpy="1.5708 0 6.7283E-16" />
-      <parent link="wrist2_Link" />
-      <child link="wrist3_Link" />
-      <axis xyz="0 0 1" />
-      <limit lower="-3.05" upper="3.05" effort="0" velocity="0" />
+      <origin xyz="0. -0.094 0." rpy="${pi/2} 0. 0."/>
+      <parent link="${prefix}wrist2_Link"/>
+      <child link="${prefix}wrist3_Link"/>
+      <axis xyz="0 0 1"/>
+      <xacro:insert_block name="wrist3_limit"/>
     </joint>
     <link name="${prefix}wrist3_Link">
@@ -212,6 +213,6 @@
       </collision>
       <inertial>
-        <origin xyz="-2.2127E-09 0.00023722 -0.018629" rpy="0 0 0" />
-        <mass value="0.13669" />
+        <origin xyz="-2.2127E-09 0.00023722 -0.018629"/>
+        <mass value="0.13669"/>
         <inertia
           ixx="6.0946E-05" ixy="9.3663E-12" ixz="-1.3841E-12"

File: aubo_description/urdf/aubo_i10_robot.urdf.xacro (robot description, xacro)
@@ -1,5 +1,5 @@
 <?xml version="1.0"?>
-<robot xmlns:xacro="http://www.ros.org/wiki/xacro" name="aubo_i5">
-  <xacro:include filename="$(find aubo_description)/urdf/aubo_i5.urdf.xacro" />
+<robot xmlns:xacro="http://www.ros.org/wiki/xacro" name="aubo_i10">
+  <xacro:include filename="$(find aubo_description)/urdf/aubo_i10.urdf.xacro" />
   <xacro:include filename="$(find aubo_description)/urdf/common.gazebo.xacro" />
   <!-- World -->
@@ -11,6 +11,6 @@
     <child link = "base_link"/>
   </joint>
-  <xacro:aubo_i5 prefix="">
+  <xacro:aubo_i10 prefix="">
     <limit lower="-3.05" upper="3.05" velocity="3.14" effort="34.0"/>
-  </xacro:aubo_i5>
+  </xacro:aubo_i10>
 </robot>

File: aubo_description/urdf/aubo_i5.urdf.xacro (robot description, xacro)
@@ -2,10 +2,4 @@
 <robot xmlns:xacro="http://www.ros.org/wiki/xacro">
   <xacro:macro name="aubo_i5" params="prefix:=''
-    *shoulder_calibration
-    *upperArm_calibration
-    *foreArm_calibration
-    *wrist1_calibration
-    *wrist2_calibration
-    *wrist3_calibration
     *wrist3_limit">
     <link name="${prefix}base_link">
@@ -39,5 +33,4 @@
       <child link="${prefix}shoulder_Link" />
       <axis xyz="0 0 1" />
-      <xacro:insert_block name="shoulder_calibration"/>
       <limit lower="-3.05" upper="3.05" velocity="2.62" effort="207.0"/>
     </joint>
@@ -72,5 +65,4 @@
       <child link="${prefix}upperArm_Link" />
       <axis xyz="0 0 1" />
-      <xacro:insert_block name="upperArm_calibration"/>
       <limit lower="-3.05" upper="3.05" velocity="2.62" effort="207.0"/>
     </joint>
@@ -105,5 +97,4 @@
       <child link="${prefix}foreArm_Link" />
       <axis xyz="0 0 1" />
-      <xacro:insert_block name="foreArm_calibration"/>
       <limit lower="-3.05" upper="3.05" velocity="2.62" effort="207.0"/>
     </joint>
@@ -138,5 +129,4 @@
       <child link="${prefix}wrist1_Link" />
       <axis xyz="0 0 1" />
-      <xacro:insert_block name="wrist1_calibration"/>
       <limit lower="-3.05" upper="3.05" velocity="3.14" effort="34.0"/>
     </joint>
@@ -171,5 +161,4 @@
       <child link="${prefix}wrist2_Link" />
       <axis xyz="0 0 1" />
-      <xacro:insert_block name="wrist2_calibration"/>
       <limit lower="-3.05" upper="3.05" velocity="3.14" effort="34.0"/>
     </joint>
@@ -204,5 +193,4 @@
       <child link="${prefix}wrist3_Link" />
       <axis xyz="0 0 1" />
-      <xacro:insert_block name="wrist3_calibration"/>
       <xacro:insert_block name="wrist3_limit"/>
     </joint>
